File: kicad_reference/example_kicad_project/stm32.kicad_sch (KiCad schematic)
At the start: 2 parts, among them U2 STM32G431C6Ux

Commit message: commit before changing more
Parts:
- added J1: Conn_01x04, symbol Connector_Generic:Conn_01x04
Connections:
- net +3V3: now also U2.20 (VREF+), J1.1 (Pin_1)
- net GND: now also J1.2 (Pin_2)
- net SWD: now reaches U2.36 (PA13)
- net SWD: now also J1.3 (Pin_3)
- net SCK: now reaches U2.37 (PA14)
- net SCK: now also J1.4 (Pin_4)
