File: kicad_schematic_parser/example_kicad_project/example_kicad_project.kicad_sch (KiCad schematic)
At the start: 0 parts

Commit message: combining labels kinda working
Other:
- added sheet labels_testing (labels_testing.kicad_sch)
Changed lines of the file:
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@@
+	)
+	(sheet
+		(at 152.4 104.14)
+		(size 15.24 15.24)
+		(fields_autoplaced yes)
+		(stroke
+			(width 0.1524)
+			(type solid)
+		)
+		(fill
+			(color 0 0 0 0.0000)
+		)
+		(property "Sheetname" "labels_testing"
+			(at 152.4 103.4284 0)
+			(effects
+				(font
+					(size 1.27 1.27)
+				)
+				(justify left bottom)
+			)
+		)
+		(property "Sheetfile" "labels_testing.kicad_sch"
+			(at 152.4 119.9646 0)
+			(effects
+				(font
+					(size 1.27 1.27)
+				)
+				(justify left top)
+			)
+		)
+		(instances
+			(project "example_kicad_project"
+				(path "/139408cf-b4ac-4ccf-8751-afbb6def1f13"
+					(page "7")
+				)
+			)
+		)
 	)
 	(sheet

Commit message: finding sheet information succesfully
Other:
- sheet labels_testing ports: added 3v3_monitor; removed none
- sheet stm32 ports: added 3v3_monitor, HW_VER; removed none
Changed lines of the file:
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@@
+			)
+		)
+		(pin "3v3_monitor" input
+			(at 167.64 109.22 0)
+			(effects
+				(font
+					(size 1.27 1.27)
+				)
+				(justify right)
 			)
 		)
@@
 			)
 		)
+		(pin "3v3_monitor" input
+			(at 133.35 60.96 0)
+			(effects
+				(font
+					(size 1.27 1.27)
+				)
+				(justify right)
+			)
+		)
+		(pin "HW_VER" input
+			(at 111.76 54.61 180)
+			(effects
+				(font
+					(size 1.27 1.27)
+				)
+				(justify left)
+			)
+		)
