File: kicad_schematic_parser/example_kicad_project/stm32.kicad_sch (KiCad schematic)
At the start: 3 parts, among them J1 Conn_01x04, U2 STM32G431C6Ux

Commit message: finding sheet information succesfully
Connections:
- net 3v3_monitor: now reaches U2.14 (PA6)
- net HW_VER: now reaches U2.24 (PB11)
Changed lines of the file:
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@@
+		)
+	)
+	(hierarchical_label "3v3_monitor"
+		(shape input)
+		(at 135.89 57.15 0)
+		(fields_autoplaced yes)
+		(effects
+			(font
+				(size 1.27 1.27)
+			)
+			(justify left)
+		)
+	)
+	(hierarchical_label "HW_VER"
+		(shape input)
+		(at 102.87 107.95 180)
+		(fields_autoplaced yes)
+		(effects
+			(font
+				(size 1.27 1.27)
+			)
+			(justify right)
 		)
 	)

Commit message: add formatting
Connections:
- net resistor_divider1/R1_2-R2_1: now reaches U2.18 (PB1)
Other:
- added sheet resistor_divider1 (resistor_divider.kicad_sch)
Changed lines of the file:
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@@
+	(wire
+		(pts
+			(xy 73.66 82.55) (xy 102.87 82.55)
+		)
+		(stroke
+			(width 0)
+			(type default)
+		)
+	)
 	(wire
 		(pts
@@
 				)
 			)
+		)
+	)
+	(sheet
+		(at 55.88 74.93)
+		(size 17.78 20.32)
+		(fields_autoplaced yes)
+		(stroke
+			(width 0.1524)
+			(type solid)
+		)
+		(fill
+			(color 0 0 0 0.0000)
+		)
+		(property "Sheetname" "resistor_divider1"
+			(at 55.88 74.2184 0)
+			(effects
+				(font
+					(size 1.27 1.27)
+				)
+				(justify left bottom)
+			)
+		)
+		(property "Sheetfile" "resistor_divider.kicad_sch"
+			(at 55.88 95.8346 0)
+			(effects
+				(font
+					(size 1.27 1.27)
+				)
+				(justify left top)
+			)
+		)
+		(pin "R1_2-R2_1" input
+			(at 73.66 82.55 0)
+			(effects
+				(font
+					(size 1.27 1.27)
+				)
+				(justify right)
+			)
+		)
+		(instances
+			(project "example_kicad_project"
+				(path "/139408cf-b4ac-4ccf-8751-afbb6def1f13/e6f5f316-cb92-4d26-9a5c-0bb6c841d4b0"
+					(page "6")
+				)
+			)
