File: kicad_schematic_parser/src/kicad_hierarchy_parser/tests/wire_connection_tests/wire_conn_test.kicad_sch (KiCad schematic)
At the start: 12 parts, among them J2 Conn_01x04, U3 NCP1117-3.3_SOT223

Commit message: committing working tests
Parts:
- renumbered C5 to C1, C7 to C2, C6 to C3, C8 to C4, J2 to J1, R3 to R1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
