File: hierachy_test/testing_hierarchy/testing_hierarchy.kicad_sch (KiCad schematic)
At the start: 0 parts

Commit message: not working yet
Other:
- removed sheet top.single_resistor
- added sheet single_resistor (single_resistor.kicad_sch)
Changed lines of the file:
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@@
     (stroke (width 0.0))
     (fill (color 0 0 0 0))
-    (property "Sheetname" "top.single_resistor" (at 115.0 45 0))
+    (property "Sheetname" "single_resistor" (at 115.0 45 0))
     (property "Sheetfile" "single_resistor.kicad_sch" (at 115.0 48 0))
   )
